Commit message: saving progress of chanages for shania

File: ros2_control_demo_description/diffbot/urdf/diffbot_description.urdf.xacro (robot description, xacro)
@@ -14,4 +14,5 @@
   <xacro:property name="caster_wheel_radius" value="0.015" />
   <xacro:property name="z_offset" value="-${base_height/2}" /> <!-- Space btw top of beam and the each joint -->
+  <link name="base_footprint" />
   <!-- Base Link -->
   <link name="${prefix}base_link">
@@ -38,4 +39,10 @@
       </inertial>
     </link>
+    <joint name="${prefix}base_link_joint" type="fixed">
+      <origin xyz="0 0 ${z_offset}" rpy="0 0 0" />
+      <parent link="base_footprint" />
+      <child link="${prefix}base_link" />
+      <axis xyz="0 0 1" />
+    </joint>
     <joint name="${prefix}left_wheel_joint" type="continuous">
       <parent link="${prefix}base_link"/>

Commit message: changes to description to fit shania

File: ros2_control_demo_description/diffbot/urdf/diffbot_description.urdf.xacro (robot description, xacro)
@@ -4,11 +4,11 @@
   <!-- Constants for robot dimensions -->
   <xacro:property name="PI" value="3.1415926535897931"/>
-  <xacro:property name="base_mass" value="0.3" /> <!-- arbitrary value for base mass -->
-  <xacro:property name="base_width" value="0.1" />
-  <xacro:property name="base_length" value="0.1" />
-  <xacro:property name="base_height" value="0.05" />
+  <xacro:property name="base_mass" value="28.0" /> <!-- arbitrary value for base mass -->
+  <xacro:property name="base_width" value="0.28" />
+  <xacro:property name="base_length" value="1.0" />
+  <xacro:property name="base_height" value="0.27393" />
   <xacro:property name="wheel_mass" value="0.3" /> <!-- arbitrary value for wheel mass -->
-  <xacro:property name="wheel_len" value="0.020" />
-  <xacro:property name="wheel_radius" value="0.015" />
+  <xacro:property name="wheel_len" value="0.06" />
+  <xacro:property name="wheel_radius" value="0.0625" />
   <xacro:property name="caster_wheel_mass" value="0.1" /> <!-- arbitrary value for caster wheel mass -->
   <xacro:property name="caster_wheel_radius" value="0.015" />
@@ -48,6 +48,6 @@
       <parent link="${prefix}base_link"/>
       <child link="${prefix}left_wheel"/>
-      <origin xyz="0 -${base_width/2} ${z_offset}" rpy="0 0 0"/>
-      <axis xyz="0 1 0"/>
+      <origin rpy="${-pi/2} 0 0" xyz="0 ${base_width/2} -${0.27393/2-wheel_radius}"/>
+      <axis rpy="0 0 0" xyz="0 0 1"/>
       <dynamics damping="0.2"/>
       <limit effort="100" velocity="1.0"/>
@@ -80,6 +80,6 @@
       <parent link="${prefix}base_link"/>
       <child link="${prefix}right_wheel"/>
-      <origin xyz="0 ${base_width/2} ${z_offset}" rpy="0 0 0"/>
-      <axis xyz="0 1 0"/>
+      <origin rpy="${-pi/2} 0 0" xyz="0 -${base_width/2} -${0.27393/2-wheel_radius}"/>
+      <axis rpy="0 0 0" xyz="0 0 1"/>
       <dynamics damping="0.2"/>
       <limit effort="100" velocity="1.0"/>

Commit message: saving progress, fixed the controller issue, made closed loop and added shania: next clean the code

File: ros2_control_demo_description/diffbot/urdf/diffbot_description.urdf.xacro (robot description, xacro)
@@ -4,17 +4,17 @@
   <!-- Constants for robot dimensions -->
   <xacro:property name="PI" value="3.1415926535897931"/>
-  <xacro:property name="base_mass" value="28.0" /> <!-- arbitrary value for base mass -->
-  <xacro:property name="base_width" value="0.28" />
+  <xacro:property name="base_mass" value="100.0" /> <!-- arbitrary value for base mass -->
+  <xacro:property name="base_width" value="0.6" />
   <xacro:property name="base_length" value="1.0" />
-  <xacro:property name="base_height" value="0.27393" />
-  <xacro:property name="wheel_mass" value="0.3" /> <!-- arbitrary value for wheel mass -->
-  <xacro:property name="wheel_len" value="0.06" />
+  <xacro:property name="base_height" value="0.3" />
+  <xacro:property name="wheel_mass" value="1.5" /> <!-- arbitrary value for wheel mass -->
+  <xacro:property name="wheel_len" value="0.05" />
   <xacro:property name="wheel_radius" value="0.0625" />
-  <xacro:property name="caster_wheel_mass" value="0.1" /> <!-- arbitrary value for caster wheel mass -->
-  <xacro:property name="caster_wheel_radius" value="0.015" />
+  <xacro:property name="caster_wheel_mass" value="0.8" /> <!-- arbitrary value for caster wheel mass -->
+  <xacro:property name="caster_wheel_radius" value="0.05" />
   <xacro:property name="z_offset" value="-${base_height/2}" /> <!-- Space btw top of beam and the each joint -->
   <link name="base_footprint" />
   <!-- Base Link -->
-  <link name="${prefix}base_link">
+ <link name="${prefix}base_link">
     <collision>
       <origin xyz="0 0 0" rpy="0 0 0"/>
@@ -48,6 +48,6 @@
       <parent link="${prefix}base_link"/>
       <child link="${prefix}left_wheel"/>
-      <origin rpy="${-pi/2} 0 0" xyz="0 ${base_width/2} -${0.27393/2-wheel_radius}"/>
-      <axis rpy="0 0 0" xyz="0 0 1"/>
+      <origin xyz="0 -${base_width/2} ${z_offset}" rpy="0 0 0"/>
+      <axis xyz="0 1 0"/>
       <dynamics damping="0.2"/>
       <limit effort="100" velocity="1.0"/>
@@ -80,6 +80,6 @@
       <parent link="${prefix}base_link"/>
       <child link="${prefix}right_wheel"/>
-      <origin rpy="${-pi/2} 0 0" xyz="0 -${base_width/2} -${0.27393/2-wheel_radius}"/>
-      <axis rpy="0 0 0" xyz="0 0 1"/>
+      <origin xyz="0 ${base_width/2} ${z_offset}" rpy="0 0 0"/>
+      <axis xyz="0 1 0"/>
       <dynamics damping="0.2"/>
       <limit effort="100" velocity="1.0"/>
